File: GuitarPedalTest.kicad_pcb (KiCad board)
At the start: 2 copper layers, 5 parts, among them U1 LM386

Commit message: Kicad test
Parts:
- moved 10uF1 33.7 mm to (106.7, 48.3)
- moved 1uF1 19.4 mm to (100.6, 48.3)
- moved 10uF2 11.4 mm to (104.1, 58.4)
Changed lines of the file:
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@@
   )
   (footprint "Capacitor_SMD:CP_Elec_3x5.3" (layer "F.Cu")
-    (at 95.02 65.31)
+    (at 104.14 58.42)
     (descr "SMT capacitor, aluminium electrolytic, 3x5.3, Cornell Dubilier Electronics ")
     (tags "Capacitor Electrolytic")
@@
   )
   (footprint "Capacitor_SMD:CP_Elec_3x5.3" (layer "F.Cu")
-    (at 82.71 55.88)
+    (at 100.56 48.26)
     (descr "SMT capacitor, aluminium electrolytic, 3x5.3, Cornell Dubilier Electronics ")
     (tags "Capacitor Electrolytic")
@@
       (effects (font (size 1 1) (thickness 0.15)))
     )
-    (fp_text user "${REFERENCE}" (at 0 0) (layer "F.Fab")
+    (fp_text user "${REFERENCE}" (at 0.4125 1.65) (layer "F.Fab")
       (effects (font (size 0.6 0.6) (thickness 0.09)))
     )
@@
   )
   (footprint "Capacitor_SMD:CP_Elec_4x5.7" (layer "F.Cu")
-    (at 75.46 60.96)
+    (at 106.68 48.26)
     (descr "SMD capacitor, aluminum electrolytic, United Chemi-Con, 4.0x5.7mm")
     (tags "capacitor electrolytic")
@@
       (effects (font (size 1 1) (thickness 0.15)))
     )
-    (fp_text user "${REFERENCE}" (at 0 0) (layer "F.Fab")
+    (fp_text user "${REFERENCE}" (at 26.14 -7.62) (layer "F.Fab")
       (effects (font (size 0.8 0.8) (thickness 0.12)))
     )
